File: PCB/MagnumFC.kicad_pcb (KiCad board)
At the start: 6 copper layers, 43.6 x 43 mm, 186 parts, among them IC1 AT7456E, J1 SM06B-SRSS-TB_LF__SN_, J10 SM04B-SRSS-TB_LF__SN_, J12 SM03B-SRSS-TB_LF__SN_, J13 SM04B-SRSS-TB_LF__SN_, J14 SM04B-SRSS-TB_LF__SN_, J2 USB4940-00-A_REVA, J3 SM03B-SRSS-TB_LF__SN_, J5 SM03B-SRSS-TB_LF__SN_, J6 SM08B-SRSS-TB_LF__SN_, J7 SM03B-SRSS-TB_LF__SN_, J8 SM03B-SRSS-TB_LF__SN_, J9 SM06B-SRSS-TB_LF__SN_, Q2 AO3400A, U1 STM32F722RETx, U10 USBLC6-2SC6, U11 AP7361C-33FGE-7, U2 BMP388, U3 NCP167BMX330TBG, U4 MP9943GQ-Z, U5 ESP32-C3, U6 ICM-42688-P, U7 W25Q256JVEIQ, U9 MP9943GQ-Z, Y1 ABM8-27.000MHZ-B2-T, Y2 C3E-40.000-10-1015-X-R, Y3 C3E-8.000-18-3030-X-R

Commit message: Update MagnumFC project files
Co-authored-by: Copilot <223556219+Copilot@users.noreply.github.com>
Other:
- board text added: "made by Poojitha S"
- board text removed: "made by Althamas Shah"
